File: HW/Star_Badge.kicad_pcb (KiCad board)
At the start: 2 copper layers, 180 x 171.6 mm, 55 parts, among them J1 AVR-ISP-6, J2 10118194-0001LF, Q1 Q_NMOS_DGS, Q2 Q_PMOS_DGS, U1 ATTINY861-15XD, U2 TPS613221ADBVT, U3 AP7363-33D-13, X1 Badgelife_sao_connector_v169b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, X2 Badgelife_sao_connector_v169b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, X3 Badgelife_sao_connector_v169b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

Commit message: Routed - net Star 2
Routing:
- net /EN_RGB4: track 0.00 -> 44.7 mm
Changed lines of the file:
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@@
     (thickness 1.6)
     (drawings 611)
-    (tracks 206)
+    (tracks 245)
     (zones 0)
     (modules 55)
@@
   (segment (start 128.75 138.25) (end 128.75 137.75) (width 0.2032) (layer B.Cu) (net 12))
   (segment (start 129.39777 144.588036) (end 129.42571 144.560096) (width 0.2032) (layer B.Cu) (net 12))
+  (segment (start 134.4 86) (end 134.6 85.53243) (width 0.2032) (layer B.Cu) (net 13))
+  (segment (start 134.9 84.991822) (end 135.2 84.4) (width 0.2032) (layer B.Cu) (net 13))
+  (segment (start 133.8 87.10617) (end 134.00531 86.69469) (width 0.2032) (layer B.Cu) (net 13))
+  (segment (start 133.59383 87.456204) (end 133.8 87.10617) (width 0.2032) (layer B.Cu) (net 13))
+  (segment (start 134.6 85.53243) (end 134.9 84.991822) (width 0.2032) (layer B.Cu) (net 13))
+  (segment (start 137.1 81.91245) (end 137.4 82.1) (width 0.2032) (layer B.Cu) (net 13))
+  (segment (start 134.00531 86.69469) (end 134.4 86) (width 0.2032) (layer B.Cu) (net 13))
+  (segment (start 133 87.9) (end 133.3 87.8) (width 0.2032) (layer B.Cu) (net 13))
+  (segment (start 131.2 87.3) (end 132 88.1) (width 0.2032) (layer B.Cu) (net 13))
+  (segment (start 137.4 82.1) (end 139.1 85.3) (width 0.2032) (layer B.Cu) (net 13))
+  (segment (start 132.6 88) (end 133 87.9) (width 0.2032) (layer B.Cu) (net 13))
+  (segment (start 133.3 87.8) (end 133.59383 87.456204) (width 0.2032) (layer B.Cu) (net 13))
+  (segment (start 135.2 84.4) (end 136 82.9) (width 0.2032) (layer B.Cu) (net 13))
+  (segment (start 136 82.9) (end 136.5 81.9) (width 0.2032) (layer B.Cu) (net 13))
+  (segment (start 136.5 81.9) (end 137.1 81.91245) (width 0.2032) (layer B.Cu) (net 13))
+  (segment (start 132 88.1) (end 132.6 88) (width 0.2032) (layer B.Cu) (net 13))
+  (segment (start 139.1 85.3) (end 139.545715 86.154285) (width 0.2032) (layer B.Cu) (net 13))
+  (segment (start 139.89295 85.80705) (end 139.545715 86.154285) (width 0.2032) (layer B.Cu) (net 13))
+  (segment (start 140.4 85.3) (end 139.89295 85.80705) (width 0.2032) (layer B.Cu) (net 13))
+  (segment (start 140.15 100.25) (end 138.85 99.6) (width 0.2032) (layer B.Cu) (net 13))
+  (segment (start 142.3 101.3) (end 140.15 100.25) (width 0.2032) (layer B.Cu) (net 13))
+  (segment (start 143 101.6) (end 142.3 101.3) (width 0.2032) (layer B.Cu) (net 13))
+  (segment (start 143.6 101.1) (end 143 101.6) (width 0.2032) (layer B.Cu) (net 13))
+  (segment (start 142.9 96.8) (end 143.5 100.5) (width 0.2032) (layer B.Cu) (net 13))
+  (segment (start 142.674348 94.525652) (end 142.9 96.8) (width 0.2032) (layer B.Cu) (net 13))
+  (segment (start 147.1 90.1) (end 142.674348 94.525652) (width 0.2032) (layer B.Cu) (net 13))
+  (segment (start 141.9 88.1) (end 142.461592 88.2) (width 0.2032) (layer B.Cu) (net 13))
+  (segment (start 142.461592 88.2) (end 143.2 88.3) (width 0.2032) (layer B.Cu) (net 13))
+  (segment (start 141.2 88) (end 141.9 88.1) (width 0.2032) (layer B.Cu) (net 13))
+  (segment (start 139.545715 86.154285) (end 140.3 87.6) (width 0.2032) (layer B.Cu) (net 13))
+  (segment (start 140.6 87.8) (end 141.2 88) (width 0.2032) (layer B.Cu) (net 13))
+  (segment (start 146.9 88.9) (end 147.2 89.322474) (width 0.2032) (layer B.Cu) (net 13))
+  (segment (start 140.3 87.6) (end 140.6 87.8) (width 0.2032) (layer B.Cu) (net 13))
+  (segment (start 138.85 99.6) (end 138.4 100.15) (width 0.2032) (layer B.Cu) (net 13))
+  (segment (start 143.2 88.3) (end 143.7 88.4) (width 0.2032) (layer B.Cu) (net 13))
+  (segment (start 143.5 100.5) (end 143.6 101.1) (width 0.2032) (layer B.Cu) (net 13))
+  (segment (start 143.7 88.4) (end 146.9 88.9) (width 0.2032) (layer B.Cu) (net 13))
+  (segment (start 147.2 89.322474) (end 147.2 89.8) (width 0.2032) (layer B.Cu) (net 13))
+  (segment (start 147.2 89.8) (end 147.1 90.1) (width 0.2032) (layer B.Cu) (net 13))
   (segment (start 102.6572 147.75) (end 106.45 147.75) (width 0.508) (layer B.Cu) (net 15))
   (segment (start 102.6572 147.75) (end 96.3 147.75) (width 0.508) (layer B.Cu) (net 15))
